File: Analog.kicad_sch (KiCad schematic)
At the start: 35 parts, among them J5 Conn_01x06, U6 MCP4725xxx-xCH, U7 MCP602, U8 MCP602

Commit message: ready for order
Parts:
- removed D3, D4, D5, D6: CG060312G, Diode_SMD:D_0603_1608Metric_Pad1.05x0.95mm_HandSolder, symbol Diode:ESD5Zxx
Connections:
- net +5V renamed +5VA
Other:
- note removed: "ESD-Protection"
